Commit message: 5.15

File: src/upros_hardware/zoo_description/urdf/w2a.urdf (robot description, URDF)
Before this commit: robot zoo_two_wheel_diff, 4 links, 3 joints
Links:
- removed link dummy
- added link base_footprint
Joints:
- removed joint dummy_joint
- added joint base_footprint_joint: type fixed, parent base_footprint, child base_link
